File: MFBadge.brd (EAGLE design)
At the start: 88.9 x 50.8 mm, 0 parts

Commit message: Added images. Checking in todays work.
Routing:
- added copper zone on layer 1, net N$1
Other:
- board size 88.9 x 50.8 mm -> 63.5 x 88.9 mm

Commit message: finished!
Parts:
- added BATT1: SMTM2032.TR, PP_Connectors:SMTM2032
- added D1, D2, D3, D4: APA3010SURCK, PP_LED:APA3010
- added R1, R2, R3, R4: 100, PP_Passives:0805
- added U$1: MF_FRAMEMF_FRAME, PP_Aesthetics:MF_FRAME
Connections:
- new net 3V: BATT1.BATT+_0, BATT1.BATT+_1, R1.1, R2.1, R3.1, R4.1
- new net GND: BATT1.BATT-, D1.1, D2.1, D3.1, D4.1
- new net N$2: D1.2, R1.2
- new net N$3: D2.2, R2.2
- new net N$4: D3.2, R3.2
- new net N$5: D4.2, R4.2
Routing:
- net GND: track 0.00 -> 154.6 mm
- net 3V: track 0.00 -> 138.6 mm
- net N$3: track 0.00 -> 3.70 mm
- net N$2: track 0.00 -> 3.70 mm
- net N$4: track 0.00 -> 3.70 mm
- net N$5: track 0.00 -> 3.70 mm
Changed lines of the file:
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@@
 <rectangle x1="21.000084375" y1="40.0107125" x2="23.804496875" y2="40.02620625" layer="29"/>
 <rectangle x1="21.263484375" y1="40.02620625" x2="23.603078125" y2="40.0417" layer="29"/>
+<rectangle x1="5.08" y1="8.89" x2="58.42" y2="27.94" layer="21"/>
+<wire x1="15.24" y1="74.93" x2="15.24" y2="41.91" width="0.4064" layer="22"/>
+<wire x1="15.24" y1="41.91" x2="48.26" y2="41.91" width="0.4064" layer="22"/>
+<wire x1="48.26" y1="41.91" x2="48.26" y2="74.93" width="0.4064" layer="22"/>
+<wire x1="48.26" y1="74.93" x2="15.24" y2="74.93" width="0.4064" layer="22"/>
 </plain>
 <attributes>
@@
 </autorouter>
 <elements>
+<element name="U$1" library="PP_Aesthetics" package="MF_FRAME" value="MF_FRAMEMF_FRAME" x="59.69" y="82.55" rot="MR0">
+<attribute name="DNAME" value="Parker Dillmann" x="59.69" y="82.55" size="1.778" layer="28" rot="MR0" display="off"/>
+<attribute name="REVNUM" value="REV 0" x="59.69" y="82.55" size="1.778" layer="28" rot="MR0" display="off"/>
+</element>
+<element name="D1" library="PP_LED" package="APA3010" value="APA3010SURCK" x="31.75" y="77.47" rot="MR180"/>
+<element name="D2" library="PP_LED" package="APA3010" value="APA3010SURCK" x="50.8" y="58.42" rot="MR270"/>
+<element name="D3" library="PP_LED" package="APA3010" value="APA3010SURCK" x="31.75" y="39.37" rot="MR0"/>
+<element name="D4" library="PP_LED" package="APA3010" value="APA3010SURCK" x="12.7" y="58.42" rot="MR90"/>
+<element name="BATT1" library="PP_Connectors" package="SMTM2032" value="SMTM2032.TR" x="31.75" y="12.7" rot="MR0"/>
+<element name="R1" library="PP_Passives" package="0805" value="100" x="38.1" y="77.47" rot="MR0"/>
+<element name="R2" library="PP_Passives" package="0805" value="100" x="50.8" y="52.07" rot="MR90"/>
+<element name="R3" library="PP_Passives" package="0805" value="100" x="25.4" y="39.37" rot="MR180"/>
+<element name="R4" library="PP_Passives" package="0805" value="100" x="12.7" y="64.77" rot="MR270"/>
 </elements>
 <signals>
@@
 </polygon>
 </signal>
+<signal name="N$2">
+<contactref element="R1" pad="2"/>
+<contactref element="D1" pad="2"/>
+<wire x1="33.5" y1="77.47" x2="37.2" y2="77.47" width="0.254" layer="16"/>
+</signal>
+<signal name="N$3">
+<contactref element="R2" pad="2"/>
+<contactref element="D2" pad="2"/>
+<wire x1="50.8" y1="52.97" x2="50.8" y2="56.67" width="0.254" layer="16"/>
+</signal>
+<signal name="N$4">
+<contactref element="R3" pad="2"/>
+<contactref element="D3" pad="2"/>
+<wire x1="26.3" y1="39.37" x2="30" y2="39.37" width="0.254" layer="16"/>
+</signal>
+<signal name="N$5">
+<contactref element="R4" pad="2"/>
+<contactref element="D4" pad="2"/>
+<wire x1="12.7" y1="63.87" x2="12.7" y2="60.17" width="0.254" layer="16"/>
+</signal>
+<signal name="3V">
+<contactref element="R1" pad="1"/>
+<contactref element="BATT1" pad="BATT+_1"/>
+<contactref element="BATT1" pad="BATT+_0"/>
+<contactref element="R4" pad="1"/>
+<contactref element="R3" pad="1"/>
+<contactref element="R2" pad="1"/>
+<wire x1="18.75" y1="12.7" x2="18.75" y2="35.26" width="0.254" layer="16"/>
+<wire x1="18.75" y1="35.26" x2="22.86" y2="39.37" width="0.254" layer="16"/>
+<wire x1="22.86" y1="39.37" x2="24.5" y2="39.37" width="0.254" layer="16"/>
+<wire x1="24.5" y1="39.37" x2="24.5" y2="40.375" width="0.254" layer="16"/>
+<wire x1="24.5" y1="40.375" x2="25.4" y2="41.275" width="0.254" layer="16"/>
+<wire x1="25.4" y1="41.275" x2="48.895" y2="41.275" width="0.254" layer="16"/>
+<wire x1="48.895" y1="41.275" x2="49.53" y2="41.91" width="0.254" layer="16"/>
+<wire x1="49.53" y1="41.91" x2="49.53" y2="51.17" width="0.254" layer="16"/>
+<wire x1="49.53" y1="51.17" x2="49.53" y2="74.93" width="0.254" layer="16"/>
+<wire x1="49.53" y1="74.93" x2="48.26" y2="76.2" width="0.254" layer="16"/>
+<wire x1="48.26" y1="76.2" x2="39.37" y2="76.2" width="0.254" layer="16"/>
+<wire x1="39" y1="76.2" x2="15.24" y2="76.2" width="0.254" layer="16"/>
+<wire x1="15.24" y1="76.2" x2="13.97" y2="74.93" width="0.254" layer="16"/>
+<wire x1="13.97" y1="74.93" x2="13.97" y2="68.58" width="0.254" layer="16"/>
+<wire x1="13.97" y1="68.58" x2="12.7" y2="67.31" width="0.254" layer="16"/>
+<wire x1="12.7" y1="67.31" x2="12.7" y2="65.67" width="0.254" layer="16"/>
+<wire x1="50.8" y1="51.17" x2="49.53" y2="51.17" width="0.254" layer="16"/>
+<wire x1="39" y1="77.47" x2="39" y2="76.2" width="0.254" layer="16"/>
+<wire x1="39" y1="76.2" x2="39.37" y2="76.2" width="0.254" layer="16"/>
+<wire x1="18.75" y1="12.7" x2="44.75" y2="12.7" width="0" layer="19" extent="16-16"/>
+</signal>
+<signal name="GND">
+<contactref element="D1" pad="1"/>
+<contactref element="BATT1" pad="BATT-"/>
+<contactref element="D4" pad="1"/>
+<contactref element="D3" pad="1"/>
+<contactref element="D2" pad="1"/>
+<wire x1="30" y1="77.47" x2="30" y2="79.375" width="0.254" layer="16"/>
+<wire x1="33.5" y1="39.37" x2="33.5" y2="23.34" width="0.254" layer="16"/>
+<wire x1="33.5" y1="23.34" x2="31.75" y2="21.59" width="0.254" layer="16"/>
+<wire x1="31.75" y1="21.59" x2="31.75" y2="12.7" width="0.254" layer="16"/>
+<wire x1="30" y1="79.375" x2="13.335" y2="79.375" width="0.254" layer="16"/>
+<wire x1="13.335" y1="79.375" x2="10.16" y2="76.2" width="0.254" layer="16"/>
+<wire x1="10.16" y1="76.2" x2="10.16" y2="57.15" width="0.254" layer="16"/>
+<wire x1="10.16" y1="57.15" x2="10.64" y2="56.67" width="0.254" layer="16"/>
+<wire x1="10.64" y1="56.67" x2="12.7" y2="56.67" width="0.254" layer="16"/>
+<wire x1="33.5" y1="39.37" x2="50.8" y2="39.37" width="0.254" layer="16"/>
+<wire x1="50.8" y1="39.37" x2="53.34" y2="41.91" width="0.254" layer="16"/>
+<wire x1="53.34" y1="41.91" x2="53.34" y2="59.69" width="0.254" layer="16"/>
+<wire x1="53.34" y1="60.17" x2="53.34" y2="76.2" width="0.254" layer="16"/>
+<wire x1="53.34" y1="76.2" x2="50.165" y2="79.375" width="0.254" layer="16"/>
+<wire x1="50.165" y1="79.375" x2="30" y2="79.375" width="0.254" layer="16"/>
+<wire x1="50.8" y1="60.17" x2="53.34" y2="60.17" width="0.254" layer="16"/>
+<wire x1="53.34" y1="60.17" x2="53.34" y2="59.69" width="0.254" layer="16"/>
+</signal>
+<signal name="N$6">
+<via x="5.08" y="5.08" extent="1-16" drill="0.5"/>
+</signal>
+<signal name="N$7">
+<via x="58.42" y="5.08" extent="1-16" drill="0.5"/>
+</signal>
 </signals>
